File: uRings_SE_Assembly_Template.brd (EAGLE design)
At the start: 40 x 110.5 mm, 0 parts

Commit message: Revision C
Parts:
- added E$1, E$2: (no value), uRings_SE_Library:M2.5-HOLE
Routing:
- added copper zone on layer 1, net GND
- added copper zone on layer 16, net GND
Other:
- board text added: "2.0 mm"
- board text added: "µRings SE Assembly Template TD-URSE-C-AT 2020-01-16 tall-dog.com"
- board text removed: "µRings SE Assembly Template TD-URSE-B-AT 2018-03-29 tall-dog.com"
Changed lines of the file:
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@@
 <?xml version="1.0" encoding="utf-8"?>
 <!DOCTYPE eagle SYSTEM "eagle.dtd">
-<eagle version="8.7.1">
+<eagle version="9.5.2">
 <drawing>
 <settings>
@@
 <layer number="51" name="tDocu" color="7" fill="1" visible="yes" active="yes"/>
 <layer number="52" name="bDocu" color="7" fill="1" visible="yes" active="yes"/>
+<layer number="88" name="SimResults" color="9" fill="1" visible="no" active="no"/>
+<layer number="89" name="SimProbes" color="9" fill="1" visible="no" active="no"/>
+<layer number="90" name="Modules" color="5" fill="1" visible="no" active="no"/>
+<layer number="91" name="Nets" color="2" fill="1" visible="no" active="no"/>
+<layer number="92" name="Busses" color="1" fill="1" visible="no" active="no"/>
+<layer number="93" name="Pins" color="2" fill="1" visible="no" active="no"/>
+<layer number="94" name="Symbols" color="4" fill="1" visible="no" active="no"/>
+<layer number="95" name="Names" color="7" fill="1" visible="no" active="no"/>
+<layer number="96" name="Values" color="7" fill="1" visible="no" active="no"/>
+<layer number="97" name="Info" color="7" fill="1" visible="no" active="no"/>
+<layer number="98" name="Guide" color="6" fill="1" visible="no" active="no"/>
 </layers>
 <board>
@@
 <hole x="5.5" y="34.5" drill="3.2"/>
 <hole x="34.5" y="34.5" drill="3.2"/>
-<text x="20" y="28" size="2" layer="21" align="center">µRings SE
+<text x="20" y="28" size="2" layer="21" ratio="12" align="center">µRings SE
 Assembly Template
-TD-URSE-B-AT
-2018-03-29
+TD-URSE-C-AT
+2020-01-16
 tall-dog.com</text>
-<text x="20" y="28" size="2" layer="22" rot="MR0" align="center">µRings SE
+<text x="20" y="28" size="2" layer="22" ratio="12" rot="MR0" align="center">µRings SE
 Assembly Template
-TD-URSE-B-AT
-2018-03-29
+TD-URSE-C-AT
+2020-01-16
 tall-dog.com</text>
+<text x="20" y="46" size="3.5" layer="22" ratio="12" rot="MR0" align="center">2.0 mm</text>
+<text x="20" y="46" size="3.5" layer="21" ratio="12" align="center">2.0 mm</text>
+<wire x1="12" y1="49" x2="28" y2="49" width="0.254" layer="21"/>
+<wire x1="28" y1="49" x2="28" y2="43" width="0.254" layer="21"/>
+<wire x1="28" y1="43" x2="12" y2="43" width="0.254" layer="21"/>
+<wire x1="12" y1="43" x2="12" y2="49" width="0.254" layer="21"/>
+<wire x1="12" y1="49" x2="28" y2="49" width="0.254" layer="22"/>
+<wire x1="28" y1="49" x2="28" y2="43" width="0.254" layer="22"/>
+<wire x1="28" y1="43" x2="12" y2="43" width="0.254" layer="22"/>
+<wire x1="12" y1="43" x2="12" y2="49" width="0.254" layer="22"/>
 </plain>
 <attributes>
@@
 <param name="checkStop" value="0"/>
 <param name="checkValues" value="0"/>
+<param name="checkNames" value="1"/>
+<param name="checkWireStubs" value="1"/>
+<param name="checkPolygonWidth" value="0"/>
 <param name="useDiameter" value="13"/>
 <param name="maxErrors" value="50"/>
@@
 </autorouter>
 <elements>
+<element name="E$1" library="uRings_SE_Library" package="M2.5-HOLE" value="" x="20" y="107.5" smashed="yes"/>
+<element name="E$2" library="uRings_SE_Library" package="M2.5-HOLE" value="" x="20" y="3" smashed="yes"/>
 </elements>
 <signals>
-<signal name="S$1">
-<via x="20" y="3" extent="1-16" drill="2.75" diameter="5"/>
-</signal>
-<signal name="S$2">
-<via x="20" y="107.5" extent="1-16" drill="2.75" diameter="5"/>
+<signal name="GND">
+<polygon width="0.5" layer="1" isolate="0.5">
+<vertex x="0" y="110.5"/>
+<vertex x="40" y="110.5"/>
+<vertex x="40" y="0"/>
+<vertex x="0" y="0"/>
+</polygon>
+<polygon width="0.5" layer="16" isolate="0.5">
+<vertex x="0" y="110.5"/>
+<vertex x="40" y="110.5"/>
+<vertex x="40" y="0"/>
+<vertex x="0" y="0"/>
+</polygon>
 </signal>
 </signals>
-<errors>
-</errors>
+<mfgpreviewcolors>
+<mfgpreviewcolor name="soldermaskcolor" color="0xC8008000"/>
+<mfgpreviewcolor name="silkscreencolor" color="0xFFFEFEFE"/>
+<mfgpreviewcolor name="backgroundcolor" color="0xFF282828"/>
+<mfgpreviewcolor name="coppercolor" color="0xFFFFBF00"/>
+<mfgpreviewcolor name="substratecolor" color="0xFF786E46"/>
+</mfgpreviewcolors>
 </board>
 </drawing>

Commit message: revision D updates continued
Other:
- board text added: "EITHER SIDE UP"
- board text added: "µRings SE Assembly Template TD-URSE-D-AT 2024-08-07 tall-dog.com"
- board text removed: "µRings SE Assembly Template TD-URSE-C-AT 2020-01-16 tall-dog.com"
Changed lines of the file:
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@@
 <?xml version="1.0" encoding="utf-8"?>
 <!DOCTYPE eagle SYSTEM "eagle.dtd">
-<eagle version="9.5.2">
+<eagle version="9.6.2">
 <drawing>
 <settings>
@@
 <text x="20" y="28" size="2" layer="21" ratio="12" align="center">µRings SE
 Assembly Template
-TD-URSE-C-AT
-2020-01-16
+TD-URSE-D-AT
+2024-08-07
 tall-dog.com</text>
 <text x="20" y="28" size="2" layer="22" ratio="12" rot="MR0" align="center">µRings SE
 Assembly Template
-TD-URSE-C-AT
-2020-01-16
+TD-URSE-D-AT
+2024-08-07
 tall-dog.com</text>
 <text x="20" y="46" size="3.5" layer="22" ratio="12" rot="MR0" align="center">2.0 mm</text>
@@
 <wire x1="28" y1="43" x2="12" y2="43" width="0.254" layer="22"/>
 <wire x1="12" y1="43" x2="12" y2="49" width="0.254" layer="22"/>
+<text x="20" y="10.5" size="2.5" layer="22" ratio="12" rot="MR0" align="center">EITHER SIDE UP</text>
+<text x="20" y="10.5" size="2.5" layer="21" ratio="12" align="center">EITHER SIDE UP</text>
 </plain>
 <attributes>
