File: uRings_SE_Control_Board.brd (EAGLE design)
At the start: 40 x 110.5 mm, 34 parts, among them J1 JACK-THONKICONN, J10 JACK-THONKICONN, J2 JACK-THONKICONN, J3 JACK-THONKICONN, J4 JACK-THONKICONN, J5 JACK-THONKICONN, J6 JACK-THONKICONN, J7 JACK-THONKICONN, J8 JACK-THONKICONN, J9 JACK-THONKICONN, P1 10k, P10 10k, P2 10k, P3 10k, P4 10k, P5 10k, P6 10k, P7 10k, P8 10k, P9 10k

Commit message: Updates for Revision C
Other:
- board text added: "2019-12-14"
- board text added: "Board derived from work by Émilie Gillet of Mutable Instruments"
- board text added: "TD-URSE-C-CB"
- board text removed: "2018-03-29"
- board text removed: "Board derived from work by Olivier Gillet of Mutable Instruments"
- board text removed: "TD-URSE-B-CB"
Changed lines of the file:
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@@
 <?xml version="1.0" encoding="utf-8"?>
 <!DOCTYPE eagle SYSTEM "eagle.dtd">
-<eagle version="8.7.1">
+<eagle version="9.5.2">
 <drawing>
 <settings>
@@
 <layers>
 <layer number="1" name="Top" color="4" fill="1" visible="yes" active="yes"/>
-<layer number="2" name="Route2" color="1" fill="3" visible="no" active="no"/>
-<layer number="15" name="Route15" color="4" fill="6" visible="no" active="no"/>
 <layer number="16" name="Bottom" color="1" fill="1" visible="yes" active="yes"/>
 <layer number="17" name="Pads" color="2" fill="1" visible="yes" active="yes"/>
@@
 <wire x1="40" y1="3" x2="37" y2="0" width="0" layer="20" curve="-90"/>
 <wire x1="37" y1="110.5" x2="40" y2="107.5" width="0" layer="20" curve="-90"/>
-<text x="39" y="87.25" size="2.5" layer="22" ratio="10" rot="MR0" align="center-left">TD-URSE-B-CB</text>
-<text x="39" y="79.75" size="2.5" layer="22" ratio="10" rot="MR0" align="center-left">2018-03-29</text>
+<text x="39" y="87.25" size="2.5" layer="22" ratio="10" rot="MR0" align="center-left">TD-URSE-C-CB</text>
+<text x="39" y="79.75" size="2.5" layer="22" ratio="10" rot="MR0" align="center-left">2019-12-14</text>
 <text x="39" y="64.75" size="2.5" layer="22" ratio="10" rot="MR0" align="center-left">tall-dog.com</text>
 <text x="39" y="72.25" size="2.5" layer="22" ratio="10" rot="MR0" align="center-left">CC BY-SA 4.0</text>
@@
 <text x="39" y="94.75" size="2.5" layer="22" ratio="10" rot="MR0" align="center-left">Control Board</text>
 <text x="20" y="8.5" size="1.5" layer="22" ratio="10" rot="MR0" align="center">Board derived from work by
-Olivier Gillet of Mutable Instruments</text>
+Émilie Gillet of Mutable Instruments</text>
 <text x="7.5" y="80" size="1.4" layer="22" ratio="10" rot="MR180" align="center">BY-SA
 4.0</text>
@@
 <param name="checkStop" value="1"/>
 <param name="checkValues" value="0"/>
+<param name="checkNames" value="1"/>
+<param name="checkWireStubs" value="1"/>
+<param name="checkPolygonWidth" value="0"/>
 <param name="useDiameter" value="13"/>
 <param name="maxErrors" value="50"/>
@@
 <attribute name="NAME" x="25.25" y="104" size="1" layer="21" ratio="10" align="top-left"/>
 </element>
-<element name="HOLE2" library="uRings_SE_Library" package="M2.5-HOLE" value="HOLE" x="20" y="3"/>
-<element name="HOLE1" library="uRings_SE_Library" package="M2.5-HOLE" value="HOLE" x="20" y="107.5"/>
+<element name="HOLE2" library="uRings_SE_Library" package="M2.5-HOLE" value="HOLE" x="20" y="3" smashed="yes"/>
+<element name="HOLE1" library="uRings_SE_Library" package="M2.5-HOLE" value="HOLE" x="20" y="107.5" smashed="yes"/>
 <element name="H1" library="uRings_SE_Library" package="PTH-0.1-2X5" value="HEADER-2X5-PTH-0.1" x="7" y="98.5" smashed="yes" rot="MR0">
 <attribute name="NAME" x="7" y="101.5" size="1" layer="22" ratio="10" rot="MR0" align="bottom-center"/>
@@
 <attribute name="NAME" x="27.75" y="38.25" size="1" layer="21" ratio="10" rot="R180" align="center"/>
 </element>
-<element name="U$1" library="uRings_SE_Library" package="MARKING-CC-LOGO" value="" x="7.5" y="85.5" rot="MR0"/>
-<element name="U$2" library="uRings_SE_Library" package="MARKING-OSH-LOGO-5MM" value="" x="7.5" y="56" rot="MR0"/>
+<element name="U$1" library="uRings_SE_Library" package="MARKING-CC-LOGO" value="" x="7.5" y="85.5" smashed="yes" rot="MR0"/>
+<element name="U$2" library="uRings_SE_Library" package="MARKING-OSH-LOGO-5MM" value="" x="7.5" y="56" smashed="yes" rot="MR0"/>
 </elements>
 <signals>
@@
 </signal>
 </signals>
+<mfgpreviewcolors>
+<mfgpreviewcolor name="soldermaskcolor" color="0xC8008000"/>
+<mfgpreviewcolor name="silkscreencolor" color="0xFFFEFEFE"/>
+<mfgpreviewcolor name="backgroundcolor" color="0xFF282828"/>
+<mfgpreviewcolor name="coppercolor" color="0xFFFFBF00"/>
+<mfgpreviewcolor name="substratecolor" color="0xFF786E46"/>
+</mfgpreviewcolors>
 <errors>
 </errors>

Commit message: Cleanup and silkscreen artwork updates
Parts:
- removed U$1: (no value), uRings_SE_Library:MARKING-CC-LOGO
- removed U$2: (no value), uRings_SE_Library:MARKING-OSH-LOGO-5MM
- H1, H2, H3, H4: device uRings_SE_Library:PTH-0.1-2X5 -> uRings_SE_Library:PTH-0.1-2X5-MALE
- P1, P10, P2, P3, P4, P5, P6, P7, P8, P9: device uRings_SE_Library:POT-ALP-VERT-PS -> uRings_SE_Library:POT
Other:
- board text added: "2019-12-18"
- board text removed: "2019-12-14"
- board text removed: "BY-SA 4.0"
- board text removed: "Board derived from work by Émilie Gillet of Mutable Instruments"
- board text removed: "CC BY-SA 4.0"
- board text removed: "Control Board"
- board text removed: "open source hardware"
- board text removed: "tall-dog.com"
- board text removed: "µRings SE"

Commit message: Revision C
Other:
- board text added: "2020-02-13"
- board text removed: "2019-12-18"
Changed lines of the file:
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@@
 <setting verticaltext="up"/>
 </settings>
-<grid distance="1" unitdist="mm" unit="mm" style="lines" multiple="1" display="yes" altdistance="0.05" altunitdist="mm" altunit="mm"/>
+<grid distance="0.25" unitdist="mm" unit="mm" style="lines" multiple="1" display="yes" altdistance="0.05" altunitdist="mm" altunit="mm"/>
 <layers>
 <layer number="1" name="Top" color="4" fill="1" visible="yes" active="yes"/>
@@
 <wire x1="37" y1="110.5" x2="40" y2="107.5" width="0.127" layer="20" curve="-90"/>
 <text x="20" y="87.25" size="2" layer="22" ratio="12" rot="MR0" align="center">TD-URSE-C-CB</text>
-<text x="20" y="79.75" size="2" layer="22" ratio="12" rot="MR0" align="center">2019-12-18</text>
+<text x="20" y="79.75" size="2" layer="22" ratio="12" rot="MR0" align="center">2020-02-13</text>
 </plain>
 <attributes>
@@
 </element>
 <element name="DS1" library="uRings_SE_Library" package="LED-SPACER" value="LED-SPACER" x="11.5" y="34.5" smashed="yes">
-<attribute name="NAME" x="11.5" y="34.5" size="1" layer="21" ratio="10" rot="R180" align="center"/>
+<attribute name="NAME" x="14.25" y="31.75" size="1.25" layer="21" ratio="10" rot="R180" align="center"/>
 <attribute name="NAME" x="11.5" y="31.75" size="1" layer="51" ratio="10" rot="R180" align="center"/>
 </element>
 <element name="DS2" library="uRings_SE_Library" package="LED-SPACER" value="LED-SPACER" x="28.5" y="34.5" smashed="yes">
-<attribute name="NAME" x="28.5" y="34.5" size="1" layer="21" ratio="10" rot="R180" align="center"/>
+<attribute name="NAME" x="25.75" y="31.75" size="1.25" layer="21" ratio="10" rot="R180" align="center"/>
 <attribute name="NAME" x="28.5" y="31.75" size="1" layer="51" ratio="10" rot="R180" align="center"/>
 </element>
@@
 <wire x1="12" y1="30.5" x2="19" y2="37.5" width="0.25" layer="1"/>
 <wire x1="19" y1="37.5" x2="23" y2="41.5" width="0.25" layer="16"/>
-<via x="19" y="37.5" extent="1-16" drill="0.3"/>
+<via x="19" y="37.5" extent="1-16" drill="0.35"/>
 <wire x1="9.54" y1="28.77" x2="11.27" y2="30.5" width="0.25" layer="1"/>
 <wire x1="11.27" y1="30.5" x2="12" y2="30.5" width="0.25" layer="1"/>
@@
 <wire x1="39.5" y1="38.25" x2="39.5" y2="27.65" width="0.25" layer="1"/>
 <wire x1="38.08" y1="26.23" x2="39.5" y2="27.65" width="0.25" layer="1"/>
-<via x="16.75" y="43" extent="1-16" drill="0.3"/>
-<via x="34.75" y="43" extent="1-16" drill="0.3"/>
+<via x="16.75" y="43" extent="1-16" drill="0.35"/>
+<via x="34.75" y="43" extent="1-16" drill="0.35"/>
 </signal>
 <signal name="SW-MODE">
@@
 <wire x1="13.5" y1="36.5" x2="14.25" y2="35.75" width="0.25" layer="16"/>
 <wire x1="14.25" y1="35.75" x2="25.25" y2="35.75" width="0.25" layer="16"/>
-<via x="25.25" y="35.75" extent="1-16" drill="0.3"/>
+<via x="25.25" y="35.75" extent="1-16" drill="0.35"/>
 <wire x1="27.92" y1="28.77" x2="25.25" y2="31.44" width="0.25" layer="1"/>
 <wire x1="25.25" y1="31.44" x2="25.25" y2="35.75" width="0.25" layer="1"/>

Commit message: updates in preparation for rev D production
Parts:
- removed DS1, DS2: LED-SPACER, uRings_SE_Library:LED-SPACER
- removed H1, H2, H3, H4: HEADER-2X5-PTH-0.1, uRings_SE_Library:PTH-0.1-2X5-MALE
- added H1-H4: HEADERS-MALE, uRings_SE_Library:HEADERS-MALE
- D1, D2: value LED-DUAL-PTH -> LED-DUAL
- J1, J10, J2, J3, J4, J5, J6, J7, J8, J9: value JACK-THONKICONN -> JACK; device uRings_SE_Library:THONKICONN -> uRings_SE_Library:JACK
- P1, P10, P2, P3, P4, P5, P6, P7, P8, P9: value 10k -> B10k
- S1, S2: value SPST-PTH -> SPST
Connections:
- net A3V3: now also H1-H4.10, H1-H4.16, H1-H4.20; no longer H1.10, H2.10, H2.6
- net BRIGHT-ATT: now also H1-H4.12; no longer H2.2
- net BRIGHT-JACK: now also H1-H4.18; no longer H2.8
- net BRIGHT-POT: now also H1-H4.14; no longer H2.4
- net DAMP-ATT: now also H1-H4.15; no longer H2.5
- net DAMP-JACK: now also H1-H4.17; no longer H2.7
- net DAMP-POT: now also H1-H4.11; no longer H2.1
- net EVEN-JACK: now also H1-H4.28; no longer H3.8
- net EVEN-SW: now also H1-H4.26; no longer H3.6
- net FREQ-ATT: now also H1-H4.2; no longer H1.2
- net FREQ-JACK: now also H1-H4.8; no longer H1.8
- net FREQ-POT: now also H1-H4.4; no longer H1.4
- net FREQ-SW: now also H1-H4.6; no longer H1.6
- net GND: now also H1-H4.13, H1-H4.19, H1-H4.3, H1-H4.32, H1-H4.9; no longer H1.3, H1.9, H2.3, H2.9, H4.2
- net IN-JACK: now also H1-H4.25; no longer H3.5
- net IN-SW: now also H1-H4.21; no longer H3.1
- net LED-MODE-GRN: now also H1-H4.36; no longer H4.6
- net LED-MODE-RED: now also H1-H4.38; no longer H4.8
- net LED-POLY-GRN: now also H1-H4.40; no longer H4.10
- net LED-POLY-RED: now also H1-H4.39; no longer H4.9
- net ODD-JACK: now also H1-H4.27; no longer H3.7
- net ODD-SW: now also H1-H4.29; no longer H3.9
- net POS-ATT: now also H1-H4.22; no longer H3.2
- net POS-JACK: now also H1-H4.30; no longer H3.10
- net POS-POT: now also H1-H4.24; no longer H3.4
- net STRUCT-ATT: now also H1-H4.5; no longer H1.5
- net STRUCT-JACK: now also H1-H4.7; no longer H1.7
- net STRUCT-POT: now also H1-H4.1; no longer H1.1
- net STRUM-JACK: now also H1-H4.35; no longer H4.5
- net STRUM-SW: now also H1-H4.37; no longer H4.7
- net SW-MODE: now also H1-H4.34; no longer H4.4
- net SW-POLY: now also H1-H4.31; no longer H4.1
- net V/OCT-JACK: now also H1-H4.23; no longer H3.3
- net V/OCT-SW: now also H1-H4.33; no longer H4.3
Other:
- board text added: "2024-07-24"
- board text added: "H1"
- board text added: "H2"
- board text added: "H3"
- board text added: "H4"
- board text added: "TD-URSE-D-CB"
- board text added: "TD-URSE-D-CB 2024-07-24 tall-dog.com"
- board text added: "tall-dog.com"
- board text removed: "2020-02-13"
- board text removed: "TD-URSE-C-CB"

Commit message: revision D updates continued
Parts:
- added U$1, U$2: (no value), uRings_SE_Library:LED-SPACER
Other:
- board text added: "2024-08-07"
- board text added: "CC BY-SA 4.0"
- board text added: "Control Board"
- board text added: "USE SPACERS UNDER LEDS"
- board text added: "µRings SE"
- board text removed: "2024-07-24"
- board text removed: "TD-URSE-D-CB 2024-07-24 tall-dog.com"
Changed lines of the file:
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@@
 <layer number="48" name="Document" color="7" fill="1" visible="no" active="yes"/>
 <layer number="49" name="Reference" color="7" fill="1" visible="no" active="yes"/>
-<layer number="51" name="tDocu" color="7" fill="1" visible="no" active="yes"/>
-<layer number="52" name="bDocu" color="7" fill="1" visible="yes" active="yes"/>
+<layer number="51" name="tDocu" color="48" fill="1" visible="no" active="yes"/>
+<layer number="52" name="bDocu" color="48" fill="1" visible="no" active="yes"/>
 <layer number="88" name="SimResults" color="9" fill="1" visible="no" active="no"/>
 <layer number="89" name="SimProbes" color="9" fill="1" visible="no" active="no"/>
@@
 <wire x1="40" y1="3" x2="37" y2="0" width="0.127" layer="20" curve="-90"/>
 <wire x1="37" y1="110.5" x2="40" y2="107.5" width="0.127" layer="20" curve="-90"/>
-<text x="20" y="57.5" size="1.5" layer="22" ratio="10" rot="MR0" align="center">TD-URSE-D-CB</text>
-<text x="20" y="49.5" size="1.5" layer="22" ratio="10" rot="MR0" align="center">2024-07-24</text>
-<text x="20" y="27.5" size="1.25" layer="21" ratio="10" align="center">TD-URSE-D-CB
-2024-07-24
-tall-dog.com</text>
+<text x="20" y="80" size="1.5" layer="22" ratio="10" rot="MR0" align="center">TD-URSE-D-CB</text>
+<text x="20" y="49.5" size="1.5" layer="22" ratio="10" rot="MR0" align="center">2024-08-07</text>
+<text x="20" y="27.5" size="1.25" layer="21" ratio="10" align="center">TD-URSE-D-CB</text>
 <text x="20" y="42.5" size="1.5" layer="22" ratio="10" rot="MR0" align="center">tall-dog.com</text>
 <text x="7" y="98.5" size="1" layer="52" ratio="10" rot="MR0" align="center">H1</text>
@@
 <text x="13.75" y="27.5" size="1" layer="22" ratio="10" rot="MR90" align="bottom-center">H3</text>
 <text x="26.25" y="27.5" size="1" layer="22" ratio="10" rot="MR270" align="bottom-center">H4</text>
+<text x="7" y="39.5" size="1" layer="21" ratio="10" align="center">USE SPACERS
+UNDER LEDS</text>
+<text x="20" y="30.5" size="1" layer="51" ratio="10" align="center">USE SPACERS UNDER LEDS</text>
+<text x="19.5" y="87.5" size="1.5" layer="22" ratio="10" rot="MR0" align="center">Control Board</text>
+<text x="19.5" y="95" size="1.5" layer="22" ratio="10" rot="MR0" align="center">µRings SE</text>
+<text x="20" y="57.5" size="1.5" layer="22" ratio="10" rot="MR0" align="center">CC BY-SA 4.0</text>
 </plain>
 <attributes>
@@
 <element name="J10" library="uRings_SE_Library" package="JACK" value="JACK" x="32.5" y="4.5" smashed="yes" rot="R270">
 <attribute name="NAME" x="27.5" y="9" size="1" layer="21" ratio="10" align="top-right"/>
-<attribute name="NAME" x="36.25" y="4.5" size="1" layer="51" ratio="10" rot="R270" align="center"/>
+<attribute name="NAME" x="32.5" y="4.5" size="1" layer="51" ratio="10" rot="R270" align="center"/>
 </element>
 <element name="J1" library="uRings_SE_Library" package="JACK" value="JACK" x="7.5" y="106" smashed="yes" rot="R90">
 <attribute name="NAME" x="12.5" y="110" size="1" layer="21" ratio="10" rot="R180" align="bottom-right"/>
-<attribute name="NAME" x="3.75" y="106" size="1" layer="51" ratio="10" rot="R90" align="center"/>
+<attribute name="NAME" x="7.5" y="106" size="1" layer="51" ratio="10" rot="R90" align="center"/>
 </element>
 <element name="J9" library="uRings_SE_Library" package="JACK" value="JACK" x="7.5" y="4.5" smashed="yes" rot="R90">
 <attribute name="NAME" x="12.5" y="9" size="1" layer="21" ratio="10" rot="R180" align="bottom-right"/>
-<attribute name="NAME" x="3.75" y="4.5" size="1" layer="51" ratio="10" rot="R90" align="center"/>
+<attribute name="NAME" x="7.5" y="4.5" size="1" layer="51" ratio="10" rot="R90" align="center"/>
 </element>
 <element name="J8" library="uRings_SE_Library" package="JACK" value="JACK" x="32.5" y="17" smashed="yes" rot="R180">
 <attribute name="NAME" x="28" y="22" size="1" layer="21" ratio="10"/>
-<attribute name="NAME" x="32.5" y="13.25" size="1" layer="51" ratio="10" rot="R180" align="center"/>
+<attribute name="NAME" x="32.5" y="17" size="1" layer="51" ratio="10" rot="R180" align="center"/>
 </element>
 <element name="J7" library="uRings_SE_Library" package="JACK" value="JACK" x="20" y="17" smashed="yes" rot="R180">
 <attribute name="NAME" x="15.5" y="22" size="1" layer="21" ratio="10"/>
-<attribute name="NAME" x="20" y="13.25" size="1" layer="51" ratio="10" rot="R180" align="center"/>
+<attribute name="NAME" x="20" y="17" size="1" layer="51" ratio="10" rot="R180" align="center"/>
 </element>
 <element name="J6" library="uRings_SE_Library" package="JACK" value="JACK" x="7.5" y="17" smashed="yes" rot="R180">
 <attribute name="NAME" x="3" y="22" size="1" layer="21" ratio="10"/>
-<attribute name="NAME" x="7.5" y="13.25" size="1" layer="51" ratio="10" rot="R180" align="center"/>
+<attribute name="NAME" x="7.5" y="17" size="1" layer="51" ratio="10" rot="R180" align="center"/>
 </element>
 <element name="J5" library="uRings_SE_Library" package="JACK" value="JACK" x="7.5" y="46" smashed="yes" rot="R90">
 <attribute name="NAME" x="12.5" y="50.5" size="1" layer="21" ratio="10" rot="R180" align="bottom-right"/>
-<attribute name="NAME" x="3.75" y="46" size="1" layer="51" ratio="10" rot="R90" align="center"/>
+<attribute name="NAME" x="7.5" y="46" size="1" layer="51" ratio="10" rot="R90" align="center"/>
 </element>
 <element name="J4" library="uRings_SE_Library" package="JACK" value="JACK" x="7.5" y="61" smashed="yes" rot="R90">
 <attribute name="NAME" x="12.5" y="65.5" size="1" layer="21" ratio="10" rot="R180" align="bottom-right"/>
-<attribute name="NAME" x="3.75" y="61" size="1" layer="51" ratio="10" rot="R90" align="center"/>
+<attribute name="NAME" x="7.5" y="61" size="1" layer="51" ratio="10" rot="R90" align="center"/>
 </element>
 <element name="J3" library="uRings_SE_Library" package="JACK" value="JACK" x="7.5" y="76" smashed="yes" rot="R90">
 <attribute name="NAME" x="12.5" y="80.5" size="1" layer="21" ratio="10" rot="R180" align="bottom-right"/>
-<attribute name="NAME" x="3.75" y="76" size="1" layer="51" ratio="10" rot="R90" align="center"/>
+<attribute name="NAME" x="7.5" y="76" size="1" layer="51" ratio="10" rot="R90" align="center"/>
 </element>
 <element name="J2" library="uRings_SE_Library" package="JACK" value="JACK" x="7.5" y="91" smashed="yes" rot="R90">
 <attribute name="NAME" x="12.5" y="95.5" size="1" layer="21" ratio="10" rot="R180" align="bottom-right"/>
-<attribute name="NAME" x="3.75" y="91" size="1" layer="51" ratio="10" rot="R90" align="center"/>
+<attribute name="NAME" x="7.5" y="91" size="1" layer="51" ratio="10" rot="R90" align="center"/>
 </element>
 <element name="P9" library="uRings_SE_Library" package="POT" value="B10k" x="32.5" y="46" smashed="yes" rot="R180">
@@
 </element>
 <element name="H1-H4" library="uRings_SE_Library" package="HEADERS-MALE" value="HEADERS-MALE" x="0" y="0" smashed="yes"/>
+<element name="U$1" library="uRings_SE_Library" package="LED-SPACER" value="" x="11.5" y="34.5" smashed="yes"/>
+<element name="U$2" library="uRings_SE_Library" package="LED-SPACER" value="" x="28.5" y="34.5" smashed="yes"/>
 </elements>
 <signals>
