File: uRings_SE_Main_Board.brd (EAGLE design)
At the start: 40 x 110.5 mm, 131 parts, among them Q1 NPN-SOT23-BEC, U1 STM32F405-LQFP-64, U2 CD4051B-TSSOP-16, U3 WM8731-SSOP-28, U4 MCP6004-TSSOP-14, U5 MCP6002-MSOP-8, U6 TL072-TSSOP-8, U7 LM1117-SOT-223, U8 ZENER-SOT-23, X1 8MHz, X2 12.288MHz

Commit message: Updates for Revision C
Parts:
- removed S1, S2: SPST-EVQPA, uRings_SE_Library:BUTTON-EVQPA
- removed U$8: (no value), uRings_SE_Library:FIDUCIAL
- removed U$9: (no value), uRings_SE_Library:MARKING-OSH-LOGO-5MM
- added C49: 47u, uRings_SE_Library:ELECTRO-SMD-6.6MM
- added R48: 2.2k, uRings_SE_Library:0603-NP
- added U$100, U$4: (no value), uRings_SE_Library:MARKING-OSH-LOGO-5MM
- added U$101: (no value), uRings_SE_Library:MARKING-CC-LOGO
- C10: value 1u -> 10u; device uRings_SE_Library:0603-NP -> uRings_SE_Library:ELECTRO-SMD-4.3MM
- C11, C17: value 0.1u -> 1u
- C16, C22, C5: value 1u -> 0.1u
- C2: value 2.2u -> 0.1u
- C20, C25, C32, C4: value 0.1u -> 18p
- C21: value 18p -> 0.1u
- C23, C6: value 18p -> 1u
- C26: value 10u -> 0.1u; device uRings_SE_Library:ELECTRO-SMD-4.3MM -> uRings_SE_Library:0603-NP
- C28: value 10n -> 10u; device uRings_SE_Library:0603-NP -> uRings_SE_Library:ELECTRO-SMD-4.3MM
- C3: value 18p -> 2.2u
- C31: value 18p -> 10n
- C36: value 2.2n -> 0.1u
- C37: value 10n -> 2.2n
- C38: value 2.2n -> 10n
- C39: value 18p -> 2.2n
- C40, C7: value 10u -> 18p; device uRings_SE_Library:ELECTRO-SMD-4.3MM -> uRings_SE_Library:0603-NP
- C42: value 220p -> 10u; device uRings_SE_Library:0603-NP -> uRings_SE_Library:ELECTRO-SMD-4.3MM
- C43: value 47u -> 220p; device uRings_SE_Library:ELECTRO-SMD-6.6MM -> uRings_SE_Library:0603-NP
- C44: value 47u -> 0.1u; device uRings_SE_Library:ELECTRO-SMD-6.6MM -> uRings_SE_Library:0603-NP
- C45, C46: value 0.1u -> 47u; device uRings_SE_Library:0603-NP -> uRings_SE_Library:ELECTRO-SMD-6.6MM
- C47: value 22u -> 0.1u; device uRings_SE_Library:ELECTRO-SMD-6.6MM -> uRings_SE_Library:0603-NP
- C48: value 47u -> 22u
- C8: value 2.2u -> 10u; device uRings_SE_Library:0603-NP -> uRings_SE_Library:ELECTRO-SMD-4.3MM
- C9: value 10u -> 2.2u; device uRings_SE_Library:ELECTRO-SMD-4.3MM -> uRings_SE_Library:0603-NP
- H6: value HEADER-1X6-PTH-SHROUDED -> HEADER-1X2; device uRings_SE_Library:JST-XH-6 -> uRings_SE_Library:PTH-0.1-1X2
- R1: value 3.3M -> 10k
- R11: value 120k -> 10k
- R14: value 20k -> 120k
- R17: value 100k -> 20k
- R18: value 47k -> 100k
- R19: value 6.8k -> 47k
- R2, R3: value 10k -> 100R
- R20: value 47k -> 6.8k
- R21, R23: value 1k -> 47k
- R22, R24: value 47k -> 1k
- R26: value 6.8k -> 100k
- R27: value 47k -> 1M; device uRings_SE_Library:0603-NP -> uRings_SE_Library:1206-NP
- R28: value 100k -> 470k; device uRings_SE_Library:0603-NP -> uRings_SE_Library:1206-NP
- R29: value 1M -> 47k
- R30: value 470k -> 6.8k
- R31: value 20k -> 47k
- R33: value 47k -> 20k
- R34: value 120k -> 47k
- R36: value 180k -> 120k
- R37: value 100k -> 180k
- R4: value 2.2k -> 3.3M; device uRings_SE_Library:0603-NP -> uRings_SE_Library:1206-NP
- R40: value 180R -> 100k
- R44: value 36k -> 180R
- R45: value 6.8k -> 36k
- R46: value 4.7R -> 6.8k; device uRings_SE_Library:1206-NP -> uRings_SE_Library:0603-NP
- R47: value 2.2k -> 4.7R; device uRings_SE_Library:0603-NP -> uRings_SE_Library:1206-NP
- R6: value 36k -> 2.2k
- R7: value 10k -> 36k
- U$2: device uRings_SE_Library:MARKING-CC-LOGO -> uRings_SE_Library:FIDUCIAL
- U$5: device uRings_SE_Library:MARKING-OSH-LOGO-5MM -> uRings_SE_Library:FIDUCIAL
- U$7: device uRings_SE_Library:FIDUCIAL -> uRings_SE_Library:TALL-DOG-LOGO-INVERT
- moved U$7 40.8 mm to (26.0, 68.2), flipped to the bottom
- moved R11 31.1 mm to (34.5, 59.5)
- moved C18 31.0 mm to (6.50, 76.5), turned to 90 degrees
- moved C17 31.0 mm to (37.5, 76.8), turned to 180 degrees
- moved R1 29.2 mm to (34.5, 102.5), turned to 0 degrees
- moved U$2 28.3 mm to (37.5, 105.5), flipped to the top, turned to 0 degrees
- moved C46 28.0 mm to (30.0, 21.0), turned to 180 degrees
- moved C9 26.6 mm to (31.5, 85.5), turned to 180 degrees
- moved R2 26.4 mm to (34.5, 98.5), turned to 180 degrees
- moved R4 25.1 mm to (4.50, 94.0)
- moved C7 24.5 mm to (11.5, 87.5)
- moved R17 24.1 mm to (10.5, 55.5)
- moved R3 23.8 mm to (34.5, 96.5), turned to 180 degrees
- moved R47 23.6 mm to (30.0, 15.5), turned to 180 degrees
- moved C6 21.0 mm to (32.5, 88.5)
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Connections:
- net JTCK renamed JTCK/SWCLK
- net JTDO renamed JTDO/SWO
- net JTMS renamed JTMS/SWDIO
- removed net BOOT: R3.2, S1.A1, S1.A2, U1.60
- new net RX1: R3.2, U1.43
- new net TX1: R2.2, U1.42
- net -10V: now also C47.2, R14.1, R37.1, R48.1; no longer C46.2, R11.1, R34.1, R47.1
- net -12V: now also C36.1, C48.C, R48.2; no longer C35.1, C47.C, R47.2
- net 12V: now also C35.2, C49.A, R47.1; no longer C34.2, C48.A, R46.1
- net A3V3: now also C10.A, C12.2, C18.2, C21.2, C23.2, C34.2, R4.2; no longer C10.2, C17.2, C19.2, C20.2, C32.2, C9.A, R1.2
- net BRIGHT-CV: now also C31.2, R17.2; no longer C30.2, R16.2
- net D3V3: now also C17.2, C19.2, C2.2, C44.2, C45.A, C6.2, C8.A, R1.2, R11.2, R6.2; no longer C1.2, C12.2, C18.2, C4.2, C43.A, C45.2, C7.A, R2.2, R4.2, R7.2, S1.B1, S1.B2
- net DAMP-CV: now also C29.2, R15.2; no longer C28.2, R14.2
- net EVEN-JACK: now also R22.2; no longer R21.2
- net EVEN-OUT: now also C28.A; no longer C27.A
- net EVEN-SW: now also R25.1; no longer R24.1
- net FREQ-CV: now also C37.2, R32.2; no longer C36.2, R31.2
- net FREQ-JACK: now also R38.1; no longer R37.1
- net FREQ-SW: now also R4.1; no longer R1.1
- net GND: now also C10.C, C26.1, C27.C, C3.1, C35.1, C36.2, C4.2, C43.1, C44.1, C45.C, C46.C, C47.1, C48.A, C49.C, C6.1, C7.2, C8.C, C9.1, R21.1, R31.1, R46.1, R7.1, U1.60; no longer C10.1, C26.C, C3.2, C32.1, C35.2, C4.1, C42.1, C43.C, C44.C, C45.1, C46.1, C47.A, C48.C, C6.2, C7.C, C8.1, C9.C, H6.1, R20.1, R27.1, R3.1, R45.1, R6.1, S2.A1, S2.A2
- net I2C-SCL: now also R5.1; no longer R4.1
- net I2C-SDA: now also R6.1; no longer R5.1
- net IN: now also C42.A; no longer C41.A
- net IN-JACK: now also R45.1; no longer R44.1
- net IN-SW: now also R27.2; no longer R29.2
- net LED-MODE-GRN: now also R44.2; no longer R43.2
- net LED-MODE-RED: now also R43.2; no longer R42.2
- net LED-POLY-GRN: now also R42.2; no longer R41.2
- net LED-POLY-RED: now also R41.2; no longer R40.2
- net N$1: now also R43.1; no longer R42.1
- net N$10: now also R41.1; no longer R40.1
- net N$11: now also C4.1; no longer C3.1
- net N$12: now also C7.1; no longer C6.1
- net N$13: now also C31.1, R14.2, R17.1; no longer C30.1, R13.2, R16.1
- net N$14: now also C39.1, R34.1, R37.2, R40.2; no longer C38.1, R33.1, R36.2, R39.2
- net N$15: now also C37.1, R32.1, R35.2, R38.2; no longer C36.1, R31.1, R34.2, R37.2
- net N$16: now also C30.1, R13.2, R16.1; no longer C29.1, R12.2, R15.1
- net N$17: now also C38.1, R33.1, R36.2, R39.2; no longer C37.1, R32.1, R35.2, R38.2
- net N$18: now also C28.C, R20.1, R21.2; no longer C27.C, R19.1, R20.2
- net N$19: now also C42.C, C43.2, R46.2; no longer C41.C, C42.2, R44.2
- net N$2: now also C46.A, R47.2; no longer C44.A, R46.2
- net N$20: now also C41.C, R30.1, R31.2; no longer C40.C, R26.1, R27.2
- net N$21: now also R18.2; no longer R17.2
- net N$22: now also C25.2; no longer C23.2
- net N$23: now also C20.2; no longer C21.2
- net N$24: now also C32.1, R19.1, R20.2, R23.2; no longer C31.1, R18.1, R19.2, R22.2
- net N$25: now also C32.2, R19.2, R22.1; no longer C31.2, R18.2, R21.1
- net N$26: now also C40.1, R25.2, R29.1, R30.2; no longer C39.1, R24.2, R25.1, R26.2
- net N$27: now also C26.2, C27.A; no longer C25.2, C26.A
- net N$28: now also R7.2; no longer R6.2
- net N$29: now also C40.2, R24.1, R29.2; no longer C39.2, R23.1, R25.2
- net N$5: now also C29.1, R12.2, R15.1; no longer C28.1, R11.2, R14.1
- net N$6: now also R44.1; no longer R43.1
- net N$7: now also C9.2; no longer C8.2
- net N$8: now also C3.2; no longer C2.2
- net N$9: now also R42.1; no longer R41.1
- net NORM-PROBE: now also R26.1, R27.1; no longer R29.1, R30.1
- net ODD-JACK: now also R24.2; no longer R23.2
- net ODD-OUT: now also C41.A; no longer C40.A
- net ODD-SW: now also R23.1; no longer R22.1
- net POS-CV: now also C38.2, R33.2; no longer C37.2, R32.2
- net POS-JACK: now also R39.1; no longer R38.1
- net RESET: now also C1.2, R1.1; no longer R2.1, S2.B1, S2.B2
- net RX: now also H6.2, R3.1; no longer H6.4, U1.43
- net STRUCT-CV: now also C30.2, R16.2; no longer C29.2, R15.2
- net STRUM: now also R11.1; no longer R7.1
- net STRUM-JACK: now also R18.1; no longer R17.1
- net STRUM-SW: now also R26.2; no longer R28.2
- net TX: now also H6.1, R2.1; no longer H6.5, U1.42
- net V/OCT-CV: now also C39.2, R34.2; no longer C38.2, R33.2
- net V/OCT-JACK: now also R40.1; no longer R39.1
- net V/OCT-SW: now also R28.2; no longer R30.2
Routing:
- net BOOT: track 20.8 -> 0.00 mm
- net D3V3: track 223.9 -> 208.5 mm, vias 9 -> 11
- net TX1: track 0.00 -> 15.3 mm, vias 0 -> 2
- net RX1: track 0.00 -> 12.3 mm, vias 0 -> 2
- net RX: track 13.7 -> 2.80 mm, vias 1 -> 0
- net GND: track 0.00 -> 10.0 mm, vias 440 -> 420
- net A3V3: track 169.1 -> 160.2 mm
- net TX: track 11.7 -> 2.80 mm, vias 1 -> 0
- net JTDI: track 8.36 -> 15.8 mm
- net RESET: track 43.6 -> 37.6 mm, vias 1 -> 2
- net JTDO/SWO: track 11.4 -> 16.8 mm
- net JTCK/SWCLK: track 12.2 -> 15.4 mm
- net JTMS/SWDIO: track 19.4 -> 21.8 mm
- net STRUM-SW: track 16.5 -> 18.2 mm
- net N$16: track 10.4 -> 8.74 mm
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Other:
- board text added: "2019-12-14"
- board text added: "Board derived from work by Émilie Gillet of Mutable Instruments"
- board text added: "MAIN BOARD"
- board text added: "SWD/JTAG"
- board text added: "TD-URSE-C 2019-12-14 tall-dog.com"
- board text added: "TD-URSE-C-MB"
- board text added: "tall-dog.com"
- board text removed: "2018-03-29"
- board text removed: "BOOT"
- board text removed: "Board derived from work by Olivier Gillet of Mutable Instruments"
- board text removed: "FTDI"
- board text removed: "JTAG"
- board text removed: "RESET"
- board text removed: "TD-URSE-B 2018-03-29 tall-dog.com"
- board text removed: "TD-URSE-B-MB"
- board text removed: "µRings_SE"

Commit message: Cleanup and silkscreen artwork updates
Parts:
- removed U$100: (no value), uRings_SE_Library:MARKING-OSH-LOGO-5MM
- removed U$101: (no value), uRings_SE_Library:MARKING-CC-LOGO
- added U$10: (no value), uRings_SE_Library:LOGO-REV
- added U$11: (no value), uRings_SE_Library:LOGO-QC
- added U$8: (no value), uRings_SE_Library:LOGO-OSHW
- added U$9: (no value), uRings_SE_Library:LOGO-TD
- H1, H2, H3, H4: device uRings_SE_Library:PTH-0.1-2X5-FLIP -> uRings_SE_Library:PTH-0.1-2X5-FEMALE
- U$1: device uRings_SE_Library:MARKING-CC-BY-SA-4.0 -> uRings_SE_Library:LOGO-PN
- U$3: device uRings_SE_Library:MARKING-CC-LOGO -> uRings_SE_Library:LOGO-CC
- U$4: device uRings_SE_Library:MARKING-OSH-LOGO-5MM -> uRings_SE_Library:LOGO-OSH
- U$7: device uRings_SE_Library:TALL-DOG-LOGO-INVERT -> uRings_SE_Library:LOGO-SN
- moved U$3 55.7 mm to (7.00, 48.0), flipped to the bottom
- moved U$4 42.7 mm to (7.00, 60.0), flipped to the bottom
- moved U$1 37.3 mm to (3.50, 83.5), flipped to the bottom, turned to 90 degrees
- moved U$7 23.8 mm to (26.0, 44.5)
Other:
- board text added: "TD-URSE-C-MB 2019-12-18"
- board text removed: "2019-12-14"
- board text removed: "BY-SA 4.0"
- board text removed: "MAIN BOARD"
- board text removed: "SN"
- board text removed: "TALL-DOG.COM"
- board text removed: "TD-URSE-C 2019-12-14 tall-dog.com"
- board text removed: "TD-URSE-C-MB"
- board text removed: "open source hardware"
- board text removed: "tall-dog.com"
- board text removed: "µRings SE"

Commit message: updates in preparation for rev D production
Parts:
- removed H1, H2, H3, H4: HEADER-2X5-PTH-0.1-FLIP, uRings_SE_Library:PTH-0.1-2X5-FEMALE
- added H1-H4: HEADERS-FEMALE, uRings_SE_Library:HEADERS-FEMALE
- added JP1: JUMPER-3, uRings_SE_Library:JUMPER-3
- D1: value DIODE-DUAL-SOT-23 -> DIODE-DUAL
- D2, D3: value DIODE-SOD123 -> DIODE
- H5: value HEADER-2X5-PTH-0.05-SHROUDED -> JTAG/SWD
- H6: value HEADER-1X2 -> SERIAL; device uRings_SE_Library:PTH-0.1-1X2 -> uRings_SE_Library:SERIAL
- H7: value HEADER-2X5-PTH-0.1-SHROUDED -> POWER
- Q1: value NPN-SOT23-BEC -> NPN
- U1: value STM32F405-LQFP-64 -> STM32F405
- U2: value CD4051B-TSSOP-16 -> CD4051B
- U3: value WM8731-SSOP-28 -> SSM2603; device uRings_SE_Library:SSOP-28 -> uRings_SE_Library:QFN-28
- U4: value MCP6004-TSSOP-14 -> MCP6004
- U5: value MCP6002-MSOP-8 -> MCP6002
- U6: value TL072-TSSOP-8 -> TL072
- U7: value LM1117-SOT-223 -> LM1117
- U8: value ZENER-SOT-23 -> ZENER
- X1: value 8MHz -> 8M
- X2: value 12.288MHz -> 12.288M
- turned H6 to 0 degrees
- turned U3 to 225 degrees
Connections:
- removed net FREQ-SW: H1.6, R4.1
- new net MUTE: JP1.2, U3.25
- new net N$30: H1-H4.6, R4.1
- net A3V3: now also H1-H4.10, H1-H4.16, H1-H4.20, U3.12, U3.18; no longer H1.10, H2.10, H2.6, U3.14, U3.8
- net BRIGHT-ATT: now also H1-H4.12; no longer H2.2
- net BRIGHT-JACK: now also H1-H4.18; no longer H2.8
- net BRIGHT-POT: now also H1-H4.14; no longer H2.4
- net D3V3: now also JP1.1, U3.3, U3.5; no longer U3.1, U3.27
- net DAMP-ATT: now also H1-H4.15; no longer H2.5
- net DAMP-JACK: now also H1-H4.17; no longer H2.7
- net DAMP-POT: now also H1-H4.11; no longer H2.1
- net EVEN-JACK: now also H1-H4.28; no longer H3.8
- net EVEN-OUT: now also U3.17; no longer U3.13
- net EVEN-SW: now also H1-H4.26; no longer H3.6
- net FREQ-ATT: now also H1-H4.2; no longer H1.2
- net FREQ-JACK: now also H1-H4.8; no longer H1.8
- net FREQ-POT: now also H1-H4.4; no longer H1.4
- net GND: now also H1-H4.13, H1-H4.19, H1-H4.3, H1-H4.32, H1-H4.9, JP1.3, U3.19, U3.26, U3.29, U3.4; no longer H1.3, H1.9, H2.3, H2.9, H4.2, U3.11, U3.21, U3.22, U3.28
- net I2C-SCL: now also U3.28; no longer U3.24
- net I2C-SDA: now also U3.27; no longer U3.23
- net I2S-LRCK: now also U3.11, U3.9; no longer U3.5, U3.7
- net I2S-SCK: now also U3.7; no longer U3.3
- net I2S-SIN: now also U3.10; no longer U3.6
- net I2S-SOUT: now also U3.8; no longer U3.4
- net IN: now also U3.23; no longer U3.19
- net IN-JACK: now also H1-H4.25; no longer H3.5
- net IN-SW: now also H1-H4.21; no longer H3.1
- net LED-MODE-GRN: now also H1-H4.36; no longer H4.6
- net LED-MODE-RED: now also H1-H4.38; no longer H4.8
- net LED-POLY-GRN: now also H1-H4.40; no longer H4.10
- net LED-POLY-RED: now also H1-H4.39; no longer H4.9
- net N$22: now also U3.1; no longer U3.25
- net N$23: now also U3.2; no longer U3.26
- net N$27: now also U3.20; no longer U3.16
- net N$28: now also U3.24; no longer U3.20
- net ODD-JACK: now also H1-H4.27; no longer H3.7
- net ODD-OUT: now also U3.16; no longer U3.12
- net ODD-SW: now also H1-H4.29; no longer H3.9
- net POS-ATT: now also H1-H4.22; no longer H3.2
- net POS-JACK: now also H1-H4.30; no longer H3.10
- net POS-POT: now also H1-H4.24; no longer H3.4
- net RX: now also H6.RX; no longer H6.2
- net STRUCT-ATT: now also H1-H4.5; no longer H1.5
- net STRUCT-JACK: now also H1-H4.7; no longer H1.7
- net STRUCT-POT: now also H1-H4.1; no longer H1.1
- net STRUM-JACK: now also H1-H4.35; no longer H4.5
- net STRUM-SW: now also H1-H4.37; no longer H4.7
- net SW-MODE: now also H1-H4.34; no longer H4.4
- net SW-POLY: now also H1-H4.31; no longer H4.1
- net TX: now also H6.TX; no longer H6.1
- net V/OCT-JACK: now also H1-H4.23; no longer H3.3
- net V/OCT-SW: now also H1-H4.33; no longer H4.3
Routing:
- net MUTE: track 0.00 -> 16.5 mm, vias 0 -> 2
- net GND: track 10.0 -> 24.0 mm, vias 420 -> 411
- net N$30: track 0.00 -> 6.41 mm
- net FREQ-SW: track 6.38 -> 0.00 mm
- net I2S-LRCK: track 35.4 -> 29.7 mm, vias 2 -> 4
- net I2S-SIN: track 27.9 -> 22.2 mm
- net I2C-SCL: track 18.8 -> 23.4 mm
- net D3V3: track 208.5 -> 213.1 mm, vias 11 -> 10
- net I2C-SDA: track 19.9 -> 24.4 mm
- net I2S-SOUT: track 20.5 -> 17.7 mm
- net EVEN-OUT: track 16.1 -> 18.7 mm
- net I2S-SCK: track 26.5 -> 24.3 mm
- net ODD-OUT: track 47.4 -> 49.5 mm
- net N$23: track 7.55 -> 9.55 mm
- net IN: track 43.1 -> 41.2 mm
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Other:
- board text added: "0"
- board text added: "1"
- board text added: "H1"
- board text added: "H2"
- board text added: "H3"
- board text added: "H4"
- board text added: "TD-URSE-D-MB 2024-07-24"
- board text removed: "TD-URSE-C-MB 2019-12-18"

Commit message: revision D updates continued
Other:
- board text added: "TD-URSE-D-MB 2024-07-30"
- board text removed: "TD-URSE-D-MB 2024-07-24"
Changed lines of the file:
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@@
 <layer number="49" name="Reference" color="7" fill="1" visible="no" active="yes"/>
 <layer number="51" name="tDocu" color="48" fill="1" visible="no" active="yes"/>
-<layer number="52" name="bDocu" color="7" fill="1" visible="no" active="yes"/>
+<layer number="52" name="bDocu" color="48" fill="1" visible="no" active="yes"/>
 <layer number="88" name="SimResults" color="9" fill="1" visible="no" active="no"/>
 <layer number="89" name="SimProbes" color="9" fill="1" visible="no" active="no"/>
@@
 <wire x1="35.65" y1="76.75" x2="36.1" y2="76.75" width="0.127" layer="21"/>
 <text x="1" y="105.5" size="1.3" layer="21" ratio="12" align="center-left">TD-URSE-D-MB
-2024-07-24</text>
+2024-07-30</text>
 <text x="38.75" y="54" size="1.5" layer="21" ratio="12" rot="R270" align="center-left">0</text>
 <text x="38.75" y="59" size="1.5" layer="21" ratio="12" rot="R90" align="center-left">1</text>
@@
 <element name="H6" library="uRings_SE_Library" package="SERIAL" value="SERIAL" x="38" y="97.5" smashed="yes" rot="MR0">
 <attribute name="NAME" x="38" y="94.6" size="1" layer="22" ratio="10" rot="MR180" align="bottom-center"/>
+<attribute name="NAME" x="38" y="97.5" size="1" layer="52" ratio="10" rot="MR270" align="center"/>
 </element>
 <element name="U$1" library="uRings_SE_Library" package="LOGO-PN" value="" x="3.5" y="83.5" smashed="yes" rot="MR90"/>
