File: uRings_SE_Main_Board.sch (EAGLE design)
At the start: 123 parts, among them Q1 NPN-SOT23-BEC, U1 STM32F405-LQFP-64, U2 CD4051B-TSSOP-16, U3 WM8731-SSOP-28, U4 MCP6004-TSSOP-14, U5 MCP6002-MSOP-8, U6 TL072-TSSOP-8, U7 LM1117-SOT-223, U8 ZENER-SOT-23, X1 8MHz, X2 12.288MHz

Commit message: Updates for Revision C
Parts:
- removed S1, S2: SPST-EVQPA, uRings_SE_Library:SPST-EVQPA
- added C49: 47u, uRings_SE_Library:CAP-P-6.6MM
- added R48: 2.2k, uRings_SE_Library:RESISTOR-0603
- C10: value 1u -> 10u; device uRings_SE_Library:CAP-NP-0603 -> uRings_SE_Library:CAP-P-4.3MM
- C11, C17: value 0.1u -> 1u
- C16, C22, C5: value 1u -> 0.1u
- C2: value 2.2u -> 0.1u
- C20, C25, C32, C4: value 0.1u -> 18p
- C21: value 18p -> 0.1u
- C23, C6: value 18p -> 1u
- C26: value 10u -> 0.1u; device uRings_SE_Library:CAP-P-4.3MM -> uRings_SE_Library:CAP-NP-0603
- C28: value 10n -> 10u; device uRings_SE_Library:CAP-NP-0603 -> uRings_SE_Library:CAP-P-4.3MM
- C3: value 18p -> 2.2u
- C31: value 18p -> 10n
- C36: value 2.2n -> 0.1u
- C37: value 10n -> 2.2n
- C38: value 2.2n -> 10n
- C39: value 18p -> 2.2n
- C40, C7: value 10u -> 18p; device uRings_SE_Library:CAP-P-4.3MM -> uRings_SE_Library:CAP-NP-0603
- C42: value 220p -> 10u; device uRings_SE_Library:CAP-NP-0603 -> uRings_SE_Library:CAP-P-4.3MM
- C43: value 47u -> 220p; device uRings_SE_Library:CAP-P-6.6MM -> uRings_SE_Library:CAP-NP-0603
- C44: value 47u -> 0.1u; device uRings_SE_Library:CAP-P-6.6MM -> uRings_SE_Library:CAP-NP-0603
- C45, C46: value 0.1u -> 47u; device uRings_SE_Library:CAP-NP-0603 -> uRings_SE_Library:CAP-P-6.6MM
- C47: value 22u -> 0.1u; device uRings_SE_Library:CAP-P-6.6MM -> uRings_SE_Library:CAP-NP-0603
- C48: value 47u -> 22u
- C8: value 2.2u -> 10u; device uRings_SE_Library:CAP-NP-0603 -> uRings_SE_Library:CAP-P-4.3MM
- C9: value 10u -> 2.2u; device uRings_SE_Library:CAP-P-4.3MM -> uRings_SE_Library:CAP-NP-0603
- H6: value HEADER-1X6-PTH-SHROUDED -> HEADER-1X2; device uRings_SE_Library:HEADER-1X6-PTH-SHROUDED -> uRings_SE_Library:HEADER-1X2
- R1: value 3.3M -> 10k
- R11: value 120k -> 10k
- R14: value 20k -> 120k
- R17: value 100k -> 20k
- R18: value 47k -> 100k
- R19: value 6.8k -> 47k
- R2, R3: value 10k -> 100R
- R20: value 47k -> 6.8k
- R21, R23: value 1k -> 47k
- R22, R24: value 47k -> 1k
- R26: value 6.8k -> 100k
- R27: value 47k -> 1M; device uRings_SE_Library:RESISTOR-0603 -> uRings_SE_Library:RESISTOR-1206
- R28: value 100k -> 470k; device uRings_SE_Library:RESISTOR-0603 -> uRings_SE_Library:RESISTOR-1206
- R29: value 1M -> 47k
- R30: value 470k -> 6.8k
- R31: value 20k -> 47k
- R33: value 47k -> 20k
- R34: value 120k -> 47k
- R36: value 180k -> 120k
- R37: value 100k -> 180k
- R4: value 2.2k -> 3.3M; device uRings_SE_Library:RESISTOR-0603 -> uRings_SE_Library:RESISTOR-1206
- R40: value 180R -> 100k
- R44: value 36k -> 180R
- R45: value 6.8k -> 36k
- R46: value 4.7R -> 6.8k; device uRings_SE_Library:RESISTOR-1206 -> uRings_SE_Library:RESISTOR-0603
- R47: value 2.2k -> 4.7R; device uRings_SE_Library:RESISTOR-0603 -> uRings_SE_Library:RESISTOR-1206
- R6: value 36k -> 2.2k
- R7: value 10k -> 36k
Connections:
- net JTCK renamed JTCK/SWCLK
- net JTDO renamed JTDO/SWO
- net JTMS renamed JTMS/SWDIO
- removed net BOOT: R3.2, S1.1, U1.BOOT0
- new net RX1: R3.2, U1.PA10
- new net TX1: R2.2, U1.PA9
- net -10V: now also C47.2, R14.1, R37.1, R48.1; no longer C46.2, R11.1, R34.1, R47.1
- net -12V: now also C36.1, C48.NEG, R48.2; no longer C35.1, C47.NEG, R47.2
- net 12V: now also C35.2, C49.POS, R47.1; no longer C34.2, C48.POS, R46.1
- net A3V3: now also C10.POS, C12.2, C18.2, C21.2, C23.2, C34.2, R4.2; no longer C10.2, C17.2, C19.2, C20.2, C32.2, C9.POS, R1.2
- net BRIGHT-CV: now also C31.2, R17.2; no longer C30.2, R16.2
- net D3V3: now also C17.2, C19.2, C2.2, C44.2, C45.POS, C6.2, C8.POS, R1.2, R11.2, R6.2; no longer C1.2, C12.2, C18.2, C4.2, C43.POS, C45.2, C7.POS, R2.2, R4.2, R7.2, S1.2
- net DAMP-CV: now also C29.2, R15.2; no longer C28.2, R14.2
- net EVEN-JACK: now also R22.2; no longer R21.2
- net EVEN-OUT: now also C28.POS; no longer C27.POS
- net EVEN-SW: now also R25.1; no longer R24.1
- net FREQ-CV: now also C37.2, R32.2; no longer C36.2, R31.2
- net FREQ-JACK: now also R38.1; no longer R37.1
- net FREQ-SW: now also R4.1; no longer R1.1
- net GND: now also C10.NEG, C26.1, C27.NEG, C3.1, C35.1, C36.2, C4.2, C43.1, C44.1, C45.NEG, C46.NEG, C47.1, C48.POS, C49.NEG, C6.1, C7.2, C8.NEG, C9.1, R21.1, R31.1, R46.1, R7.1, U1.BOOT0; no longer C10.1, C26.NEG, C3.2, C32.1, C35.2, C4.1, C42.1, C43.NEG, C44.NEG, C45.1, C46.1, C47.POS, C48.NEG, C6.2, C7.NEG, C8.1, C9.NEG, H6.1, R20.1, R27.1, R3.1, R45.1, R6.1, S2.1
- net I2C-SCL: now also R5.1; no longer R4.1
- net I2C-SDA: now also R6.1; no longer R5.1
- net IN: now also C42.POS; no longer C41.POS
- net IN-JACK: now also R45.1; no longer R44.1
- net IN-SW: now also R27.2; no longer R29.2
- net LED-MODE-GRN: now also R44.2; no longer R43.2
- net LED-MODE-RED: now also R43.2; no longer R42.2
- net LED-POLY-GRN: now also R42.2; no longer R41.2
- net LED-POLY-RED: now also R41.2; no longer R40.2
- net N$1: now also R43.1; no longer R42.1
- net N$10: now also R41.1; no longer R40.1
- net N$11: now also C4.1; no longer C3.1
- net N$12: now also C7.1; no longer C6.1
- net N$13: now also C31.1, R14.2, R17.1; no longer C30.1, R13.2, R16.1
- net N$14: now also C39.1, R34.1, R37.2, R40.2; no longer C38.1, R33.1, R36.2, R39.2
- net N$15: now also C37.1, R32.1, R35.2, R38.2; no longer C36.1, R31.1, R34.2, R37.2
- net N$16: now also C30.1, R13.2, R16.1; no longer C29.1, R12.2, R15.1
- net N$17: now also C38.1, R33.1, R36.2, R39.2; no longer C37.1, R32.1, R35.2, R38.2
- net N$18: now also C28.NEG, R20.1, R21.2; no longer C27.NEG, R19.1, R20.2
- net N$19: now also C42.NEG, C43.2, R46.2; no longer C41.NEG, C42.2, R44.2
- net N$2: now also C46.POS, R47.2; no longer C44.POS, R46.2
- net N$20: now also C41.NEG, R30.1, R31.2; no longer C40.NEG, R26.1, R27.2
- net N$21: now also R18.2; no longer R17.2
- net N$22: now also C25.2; no longer C23.2
- net N$23: now also C20.2; no longer C21.2
- net N$24: now also C32.1, R19.1, R20.2, R23.2; no longer C31.1, R18.1, R19.2, R22.2
- net N$25: now also C32.2, R19.2, R22.1; no longer C31.2, R18.2, R21.1
- net N$26: now also C40.1, R25.2, R29.1, R30.2; no longer C39.1, R24.2, R25.1, R26.2
- net N$27: now also C26.2, C27.POS; no longer C25.2, C26.POS
- net N$28: now also R7.2; no longer R6.2
- net N$29: now also C40.2, R24.1, R29.2; no longer C39.2, R23.1, R25.2
- net N$5: now also C29.1, R12.2, R15.1; no longer C28.1, R11.2, R14.1
- net N$6: now also R44.1; no longer R43.1
- net N$7: now also C9.2; no longer C8.2
- net N$8: now also C3.2; no longer C2.2
- net N$9: now also R42.1; no longer R41.1
- net NORM-PROBE: now also R26.1, R27.1; no longer R29.1, R30.1
- net ODD-JACK: now also R24.2; no longer R23.2
- net ODD-OUT: now also C41.POS; no longer C40.POS
- net ODD-SW: now also R23.1; no longer R22.1
- net POS-CV: now also C38.2, R33.2; no longer C37.2, R32.2
- net POS-JACK: now also R39.1; no longer R38.1
- net RESET: now also C1.2, R1.1; no longer R2.1, S2.2
- net RX: now also H6.2, R3.1; no longer H6.4, U1.PA10
- net STRUCT-CV: now also C30.2, R16.2; no longer C29.2, R15.2
- net STRUM: now also R11.1; no longer R7.1
- net STRUM-JACK: now also R18.1; no longer R17.1
- net STRUM-SW: now also R26.2; no longer R28.2
- net TX: now also H6.1, R2.1; no longer H6.5, U1.PA9
- net V/OCT-CV: now also C39.2, R34.2; no longer C38.2, R33.2
- net V/OCT-JACK: now also R40.1; no longer R39.1
- net V/OCT-SW: now also R28.2; no longer R30.2
Other:
- note added: "C"
- note added: "Licensed: CC BY-SA 4.0 Board derived from work by Émilie Gillet of Mutable Instruments"
- note removed: "B"
- note removed: "Licensed: CC BY-SA 4.0 Board derived from work by Olivier Gillet of Mutable Instruments"
- moved on the sheet: C1, C11, C12, C13, C14, C15, C16, C19, C2, C20, C21, C22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

Commit message: updates in preparation for rev D production
Parts:
- removed H1, H2, H3, H4: HEADER-2X5-PTH-0.1-FLIP, uRings_SE_Library:HEADER-2X5-PTH-0.1-FLIP
- added H1-H4: HEADERS-FEMALE, uRings_SE_Library:HEADERS-FEMALE
- added JP1: JUMPER-3, uRings_SE_Library:JUMPER-3
- D1: value DIODE-DUAL-SOT-23 -> DIODE-DUAL; device uRings_SE_Library:DIODE-DUAL-SOT-23 -> uRings_SE_Library:DIODE-DUAL
- D2, D3: value DIODE-SOD123 -> DIODE; device uRings_SE_Library:DIODE-SOD123 -> uRings_SE_Library:DIODE
- H5: value HEADER-2X5-PTH-0.05-SHROUDED -> JTAG/SWD; device uRings_SE_Library:HEADER-2X5-PTH-0.05-SHROUDED -> uRings_SE_Library:JTAG/SWD
- H6: value HEADER-1X2 -> SERIAL; device uRings_SE_Library:HEADER-1X2 -> uRings_SE_Library:SERIAL
- H7: value HEADER-2X5-PTH-0.1-SHROUDED -> POWER; device uRings_SE_Library:HEADER-2X5-PTH-0.1-SHROUDED -> uRings_SE_Library:POWER
- Q1: value NPN-SOT23-BEC -> NPN; device uRings_SE_Library:NPN-SOT23-BEC -> uRings_SE_Library:NPN
- U1: value STM32F405-LQFP-64 -> STM32F405; device uRings_SE_Library:STM32F405-LQFP-64 -> uRings_SE_Library:STM32F405
- U2: value CD4051B-TSSOP-16 -> CD4051B; device uRings_SE_Library:CD4051B-TSSOP-16 -> uRings_SE_Library:CD4051B
- U3: value WM8731-SSOP-28 -> SSM2603; device uRings_SE_Library:WM8731-SSOP-28 -> uRings_SE_Library:SSM2603
- U4: value MCP6004-TSSOP-14 -> MCP6004; device uRings_SE_Library:MCP6004-TSSOP-14 -> uRings_SE_Library:MCP6004
- U5: value MCP6002-MSOP-8 -> MCP6002; device uRings_SE_Library:MCP6002-MSOP-8 -> uRings_SE_Library:MCP6002
- U6: value TL072-TSSOP-8 -> TL072; device uRings_SE_Library:TL072-TSSOP-8 -> uRings_SE_Library:TL072
- U7: value LM1117-SOT-223 -> LM1117; device uRings_SE_Library:LM1117-SOT-223 -> uRings_SE_Library:LM1117
- U8: value ZENER-SOT-23 -> ZENER; device uRings_SE_Library:ZENER-SOT-23 -> uRings_SE_Library:ZENER
- X1: value 8MHz -> 8M; device uRings_SE_Library:CRYSTAL-ABM3 -> uRings_SE_Library:CRYSTAL
- X2: value 12.288MHz -> 12.288M; device uRings_SE_Library:CRYSTAL-ABM3 -> uRings_SE_Library:CRYSTAL
Connections:
- removed net FREQ-SW: H1.6, R4.1
- new net MUTE: JP1.2, U3.MUTE
- new net N$30: H1-H4.FREQ-SW, R4.1
- net -12V: now also U6A.NEG; no longer U6P.-
- net 12V: now also U6A.POS; no longer U6P.+
- net A3V3: now also H1-H4.A3V3, U4A.POS, U5A.POS; no longer H1.10, H2.10, H2.6, U4P.+, U5P.+
- net BRIGHT-ATT: now also H1-H4.BRIGHT-ATT; no longer H2.2
- net BRIGHT-JACK: now also H1-H4.BRIGHT-JACK; no longer H2.8
- net BRIGHT-POT: now also H1-H4.BRIGHT-POT; no longer H2.4
- net D3V3: now also H5.VCC, JP1.1; no longer H5.1
- net DAMP-ATT: now also H1-H4.DAMP-ATT; no longer H2.5
- net DAMP-JACK: now also H1-H4.DAMP-JACK; no longer H2.7
- net DAMP-POT: now also H1-H4.DAMP-POT; no longer H2.1
- net EVEN-JACK: now also H1-H4.EVEN-JACK; no longer H3.8
- net EVEN-SW: now also H1-H4.EVEN-SW; no longer H3.6
- net FREQ-ATT: now also H1-H4.FREQ-ATT; no longer H1.2
- net FREQ-JACK: now also H1-H4.FREQ-JACK; no longer H1.8
- net FREQ-POT: now also H1-H4.FREQ-POT; no longer H1.4
- net GND: now also H1-H4.GND, H5.GND, H7.GND, JP1.3, U3.PGND, U4A.IN+, U4A.NEG, U5A.IN+, U5A.NEG, U6A.IN+; no longer H1.3, H1.9, H2.3, H2.9, H4.2, H5.3, H5.5, H5.9, H7.3, H7.4, H7.5, H7.6, H7.7, H7.8, U3.HPGND, U3.MODE, U4A.+, U4P.-, U5A.+, U5P.-, U6A.+
- net I2S-LRCK: now also U3.PBLRC, U3.RECLRC; no longer U3.ADCLRC, U3.DACLRC
- net I2S-SIN: now also U3.RECDAT; no longer U3.ADCDAT
- net I2S-SOUT: now also U3.PBDAT; no longer U3.DACDAT
- net IN-JACK: now also H1-H4.IN-JACK; no longer H3.5
- net IN-SW: now also H1-H4.IN-SW; no longer H3.1
- net JTCK/SWCLK: now also H5.TCK/SWCLK; no longer H5.4
- net JTDI: now also H5.TDI; no longer H5.8
- net JTDO/SWO: now also H5.TDO/SWO; no longer H5.6
- net JTMS/SWDIO: now also H5.TMS/SWDIO; no longer H5.2
- net LED-MODE-GRN: now also H1-H4.LED-MODE-GRN; no longer H4.6
- net LED-MODE-RED: now also H1-H4.LED-MODE-RED; no longer H4.8
- net LED-POLY-GRN: now also H1-H4.LED-POLY-GRN; no longer H4.10
- net LED-POLY-RED: now also H1-H4.LED-POLY-RED; no longer H4.9
- net MUXED-POTS: now also U2.COM; no longer U2.X
- net N$100: now also H7.-12V; no longer H7.1, H7.2
- net N$101: now also H7.+12V; no longer H7.10, H7.9
- net N$13: now also U5A.IN-; no longer U5A.-
- net N$16: now also U4A.IN-; no longer U4A.-
- net N$22: now also U3.MCLK/XTI; no longer U3.XTI/MCLK
- net N$26: now also U6A.IN-; no longer U6A.-
- net ODD-JACK: now also H1-H4.ODD-JACK; no longer H3.7
- net ODD-SW: now also H1-H4.ODD-SW; no longer H3.9
- net POS-ATT: now also H1-H4.POS-ATT; no longer H3.2
- net POS-JACK: now also H1-H4.POS-JACK; no longer H3.10
- net POS-POT: now also H1-H4.POS-POT; no longer H3.4
- net RESET: now also H5.RESET; no longer H5.10
- net RX: now also H6.RX; no longer H6.2
- net STRUCT-ATT: now also H1-H4.STRUCT-ATT; no longer H1.5
- net STRUCT-JACK: now also H1-H4.STRUCT-JACK; no longer H1.7
- net STRUCT-POT: now also H1-H4.STRUCT-POT; no longer H1.1
- net STRUM-JACK: now also H1-H4.STRUM-JACK; no longer H4.5
- net STRUM-SW: now also H1-H4.STRUM-SW; no longer H4.7
- net SW-MODE: now also H1-H4.SW-MODE; no longer H4.4
- net SW-POLY: now also H1-H4.SW-POLY; no longer H4.1
- net TX: now also H6.TX; no longer H6.1
- net V/OCT-JACK: now also H1-H4.V/OCT-JACK; no longer H3.3
- net V/OCT-SW: now also H1-H4.V/OCT-SW; no longer H4.3
Other:
- note added: "TD-URSE-D-MB"
- note added: "tall-dog.com"
- note removed: "Analog"
- note removed: "C"
- note removed: "CV Scaling"
- note removed: "Main Processor"
- note removed: "N/A"
- note removed: "Supply"
- note removed: "User Interface"
- note removed: "Website: tall-dog.com"
